File: PCB/PCB_v8.brd (EAGLE design)
At the start: 46 x 26 mm, 23 parts, among them J1 USB4125-GF-A_REVA, J2 F-1X04-SIP-100-40, J3 PINHD-1X2, Q1 NMOSFET, U1 AP2112K-3.3TRG1, U2 ESP32-WROOM

Commit message: Add hardware files
Parts:
- removed C3, C4, C5: 10uF, Capacitor:CAPC1608X85
- moved R7 14.2 mm to (29.6, 20.1), turned to 270 degrees
- moved R8 7.37 mm to (27.1, 20.1)
- moved C2 2.54 mm to (24.5, 20.1)
Connections:
- net +5V: no longer C3.2, C4.2, C5.2
- net GND: no longer C3.1, C4.1, C5.1
Routing:
- net GPIO17: track 14.8 -> 51.2 mm
- net +5V: track 78.2 -> 102.5 mm, vias 1 -> 5
- net EN: track 58.1 -> 70.4 mm, vias 3 -> 1
- net GPIO32: track 13.8 -> 4.16 mm
- net GND: track 160.2 -> 152.5 mm, vias 4 -> 1
- net LED: track 7.12 -> 13.4 mm
- net +3.3V: track 55.9 -> 50.7 mm, vias 3 -> 1
- net DATA: track 24.6 -> 19.6 mm
- net D: track 27.2 -> 30.8 mm, vias 1 -> 0
- net ESP_RX: track 30.6 -> 31.7 mm
Other:
- board text added: "by Oleksii Kutuzov ESP32 LED Strip Controller v1.1"
- board text removed: "by Oleksii Kutuzov ESP32 LED Strip Controller v1.0"
