File: PCB/Schematic_v1.1_v8.sch (EAGLE design)
At the start: 23 parts, among them J1 USB4125-GF-A_REVA, J2 F-1X04-SIP-100-40, J3 PINHD-1X2, Q1 NMOSFET, U1 AP2112K-3.3TRG1, U2 ESP32-WROOM

Commit message: Add hardware files
Parts:
- removed C3, C4, C5: 10uF, Capacitor:C_CHIP-0603(1608-METRIC)
Connections:
- net +5V: no longer C3.2, C4.2, C5.2
- net GND: no longer C3.1, C4.1, C5.1
Changed lines of the file:
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@@
 <part name="SUPPLY22" library="Power_Symbols" deviceset="GND" device="" value="GND"/>
 <part name="R7" library="Resistor" deviceset="R" device="CHIP-0603(1608-METRIC)" package3d_urn="urn:adsk.eagle:package:16378565/2" technology="_" value="300-500 ohm"/>
-<part name="C3" library="Capacitor" deviceset="C" device="CHIP-0603(1608-METRIC)" package3d_urn="urn:adsk.eagle:package:16290898/2" technology="_" value="10uF"/>
-<part name="C4" library="Capacitor" deviceset="C" device="CHIP-0603(1608-METRIC)" package3d_urn="urn:adsk.eagle:package:16290898/2" technology="_" value="10uF"/>
-<part name="C5" library="Capacitor" deviceset="C" device="CHIP-0603(1608-METRIC)" package3d_urn="urn:adsk.eagle:package:16290898/2" technology="_" value="10uF"/>
 <part name="R2" library="Resistor" deviceset="R" device="CHIP-0603(1608-METRIC)" package3d_urn="urn:adsk.eagle:package:16378565/2" technology="_" value="5.1k"/>
 </parts>
@@
 <attribute name="VALUE" x="152.4" y="130.81" size="1.778" layer="96" rot="R90"/>
 </instance>
-<instance part="SUPPLY19" gate="G$1" x="157.48" y="165.1" smashed="yes">
-<attribute name="VALUE" x="157.353" y="168.148" size="1.778" layer="96" align="bottom-center"/>
-</instance>
-<instance part="SUPPLY20" gate="G$1" x="132.08" y="167.64" smashed="yes" rot="R180">
-<attribute name="VALUE" x="132.08" y="170.18" size="1.778" layer="96" rot="R180" align="center"/>
+<instance part="SUPPLY19" gate="G$1" x="154.94" y="119.38" smashed="yes" rot="R180">
+<attribute name="VALUE" x="155.067" y="116.332" size="1.778" layer="96" rot="R180" align="bottom-center"/>
+</instance>
+<instance part="SUPPLY20" gate="G$1" x="134.62" y="116.84" smashed="yes">
+<attribute name="VALUE" x="134.62" y="114.3" size="1.778" layer="96" align="center"/>
 </instance>
 <instance part="J3" gate="G$1" x="111.76" y="172.72" smashed="yes" rot="R90">
@@
 <attribute name="NAME" x="142.24" y="111.76" size="1.778" layer="95" rot="R90" align="center"/>
 <attribute name="VALUE" x="147.32" y="111.76" size="1.778" layer="96" rot="R90" align="center"/>
-</instance>
-<instance part="C3" gate="G$1" x="143.256" y="153.924" smashed="yes" rot="R90">
-<attribute name="NAME" x="140.716" y="158.496" size="1.778" layer="95" rot="R180"/>
-<attribute name="VALUE" x="146.304" y="156.464" size="1.778" layer="96"/>
-</instance>
-<instance part="C4" gate="G$1" x="143.256" y="148.844" smashed="yes" rot="R90">
-<attribute name="NAME" x="140.716" y="153.416" size="1.778" layer="95" rot="R180"/>
-<attribute name="VALUE" x="146.304" y="151.384" size="1.778" layer="96"/>
-</instance>
-<instance part="C5" gate="G$1" x="143.256" y="159.004" smashed="yes" rot="R90">
-<attribute name="NAME" x="140.716" y="163.576" size="1.778" layer="95" rot="R180"/>
-<attribute name="VALUE" x="146.304" y="161.544" size="1.778" layer="96"/>
 </instance>
 <instance part="R2" gate="G$1" x="-38.1" y="96.52" smashed="yes">
@@
 <segment>
 <pinref part="SUPPLY20" gate="G$1" pin="GND"/>
-<wire x1="132.08" y1="165.1" x2="132.08" y2="159.004" width="0.1524" layer="91"/>
-<wire x1="132.08" y1="159.004" x2="132.08" y2="153.924" width="0.1524" layer="91"/>
-<wire x1="132.08" y1="153.924" x2="132.08" y2="149.86" width="0.1524" layer="91"/>
-<wire x1="132.08" y1="148.844" x2="132.08" y2="124.46" width="0.1524" layer="91"/>
-<wire x1="132.08" y1="124.46" x2="142.24" y2="124.46" width="0.1524" layer="91"/>
+<wire x1="134.62" y1="119.38" x2="134.62" y2="124.46" width="0.1524" layer="91"/>
+<wire x1="134.62" y1="124.46" x2="142.24" y2="124.46" width="0.1524" layer="91"/>
 <wire x1="142.24" y1="124.46" x2="142.24" y2="134.62" width="0.1524" layer="91"/>
 <pinref part="LED1" gate="A" pin="1"/>
 <label x="142.24" y="139.7" size="1.778" layer="95" rot="R90"/>
-<pinref part="C3" gate="G$1" pin="1"/>
-<wire x1="140.716" y1="153.924" x2="132.08" y2="153.924" width="0.1524" layer="91"/>
-<pinref part="C5" gate="G$1" pin="1"/>
-<wire x1="140.716" y1="159.004" x2="132.08" y2="159.004" width="0.1524" layer="91"/>
-<pinref part="C4" gate="G$1" pin="1"/>
-<wire x1="140.716" y1="148.844" x2="132.08" y2="148.844" width="0.1524" layer="91"/>
-<wire x1="132.08" y1="148.844" x2="132.08" y2="149.86" width="0.1524" layer="91"/>
-<junction x="132.08" y="159.004"/>
-<junction x="132.08" y="153.924"/>
-<junction x="132.08" y="148.844"/>
 </segment>
 </net>
@@
 <segment>
 <pinref part="SUPPLY19" gate="G$1" pin="+5V"/>
-<wire x1="157.48" y1="165.1" x2="157.48" y2="159.004" width="0.1524" layer="91"/>
-<wire x1="157.48" y1="159.004" x2="157.48" y2="153.924" width="0.1524" layer="91"/>
-<wire x1="157.48" y1="153.924" x2="157.48" y2="149.86" width="0.1524" layer="91"/>
-<wire x1="157.48" y1="148.844" x2="157.48" y2="124.46" width="0.1524" layer="91"/>
-<wire x1="157.48" y1="124.46" x2="147.32" y2="124.46" width="0.1524" layer="91"/>
+<wire x1="154.94" y1="119.38" x2="154.94" y2="124.46" width="0.1524" layer="91"/>
+<wire x1="154.94" y1="124.46" x2="147.32" y2="124.46" width="0.1524" layer="91"/>
 <wire x1="147.32" y1="124.46" x2="147.32" y2="134.62" width="0.1524" layer="91"/>
 <pinref part="LED1" gate="A" pin="3"/>
 <label x="147.32" y="139.7" size="1.778" layer="95" rot="R90"/>
-<pinref part="C3" gate="G$1" pin="2"/>
-<wire x1="148.336" y1="153.924" x2="157.48" y2="153.924" width="0.1524" layer="91"/>
-<pinref part="C5" gate="G$1" pin="2"/>
-<wire x1="148.336" y1="159.004" x2="157.48" y2="159.004" width="0.1524" layer="91"/>
-<pinref part="C4" gate="G$1" pin="2"/>
-<wire x1="148.336" y1="148.844" x2="157.48" y2="148.844" width="0.1524" layer="91"/>
-<wire x1="157.48" y1="148.844" x2="157.48" y2="149.86" width="0.1524" layer="91"/>
-<junction x="157.48" y="159.004"/>
-<junction x="157.48" y="153.924"/>
-<junction x="157.48" y="148.844"/>
 </segment>
 </net>
