File: PCB/ESP32/ESP32_PCB_v12.brd (EAGLE design)
At the start: 46 x 26 mm, 20 parts, among them J1 USB4125-GF-A_REVA, J2 F-1X04-SIP-100-40, J3 PINHD-1X2, Q1 NMOSFET, U1 AP2112K-3.3TRG1, U2 ESP32-WROOM

Commit message: Upload ESP32-C3 hardware files
Routing:
- net GND: track 152.5 -> 0.00 mm, vias 1 -> 0
- net EN: track 70.4 -> 44.7 mm
- net +5V: track 102.5 -> 81.6 mm, vias 5 -> 1
- net D: track 30.8 -> 46.1 mm
- net GPIO17: track 51.2 -> 43.2 mm
- net DATA: track 19.6 -> 15.1 mm, vias 0 -> 2
- net ESP_RX: track 31.7 -> 27.2 mm
- net LED: track 13.4 -> 17.9 mm
- net ESP_TX: track 24.1 -> 27.8 mm, vias 0 -> 1
- net GPIO0: track 17.4 -> 20.4 mm, vias 2 -> 1
- net CC: track 9.32 -> 12.3 mm
- net N$1: track 8.56 -> 11.3 mm
- net +3.3V: track 50.7 -> 53.0 mm
- net GPIO18: track 8.03 -> 9.70 mm
- net GPIO32: track 4.16 -> 4.76 mm
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Other:
- outline, holes or cut-outs redrawn
- board text added: "ESP32 LED Strip Controller v1.1 by Oleksii Kutuzov"
- board text removed: "by Oleksii Kutuzov ESP32 LED Strip Controller v1.1"
